File: attiny_pwm.kicad_pcb (KiCad board)
At the start: 2 copper layers, 45 x 42 mm, 29 parts, among them J1 PWM Output, J2 Conn_01x03_Pin, Q1 IRLZ44N, SW1 SW_Push, SW2 SW_Push, SW3 SW_Push, U1 LM2937xMP, U2 ATtiny402-SS

Commit message: erased fuckups
Parts:
- BT1: value 12VDC Input -> Battery
- J1: value PWM Output -> Screw_Terminal_01x02
- R2: value 4k7 -> 0
- RV1: value Potentiometer -> R_Potentiometer
- moved D1 13.7 mm to (164.0, 101.4), turned to -90 degrees
- moved R1 13.3 mm to (164.0, 105.7), turned to -90 degrees
- moved U1 3.80 mm to (156.5, 103.8)
Routing:
- net GND: track 61.6 -> 49.1 mm
- net 5V: track 112.1 -> 108.4 mm
- net /Vin: track 68.6 -> 69.5 mm
