File: attiny_pwm.kicad_sch (KiCad schematic)
At the start: 28 parts, among them J1 Screw_Terminal_01x02, J2 Conn_01x03_Pin, Q1 IRLZ44N, SW1 SW_Push, SW2 SW_Push, SW3 SW_Push, U1 LM2937xMP, U2 ATtiny402-SS

Commit message: erased fuckups
Parts:
- R2: value 4k7 -> 0
Changed lines of the file:
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@@
 			)
 		)
-		(property "Value" "4k7"
+		(property "Value" "0"
 			(at 87.63 105.156 0)
 			(effects
